Commit message: ar track

File: src/my_r2d2/urdf/r2d2.urdf.xacro (robot description, xacro)
@@ -231,5 +231,5 @@
     <parent link="box"/>
     <child link="lense"/>
-    <origin xyz="0 0 0"/>
+    <origin xyz="0 0 0" rpy="0 0 0" />
   </joint>
 <link name="base_footprint">
@@ -240,3 +240,11 @@
     <origin xyz="0 0 0.48"/>
   </joint>
+<link name="eye">
+<origin xyz="0 0 0" rpy="0 0 0" />
+  </link>
+<joint name="eye_lense" type="fixed">
+    <parent link="lense"/>
+    <child link="eye"/>
+    <origin xyz="0 0 0" rpy="0 ${pi/2} ${pi/2}"/>
+  </joint>
 </robot>

Commit message: Lab 6 - Sensor

File: src/my_r2d2/urdf/r2d2.urdf.xacro (robot description, xacro)
@@ -246,5 +246,5 @@
     <parent link="lense"/>
     <child link="eye"/>
-    <origin xyz="0 0 0" rpy="0 ${pi/2} ${pi/2}"/>
+    <origin xyz="0 0 0" rpy="-${pi/2} 0 -${pi/2}"/>
   </joint>
 </robot>

Commit message: Review

File: src/my_r2d2/urdf/r2d2.urdf.xacro (robot description, xacro)
@@ -228,7 +228,8 @@
     <xacro:default_inertial mass="1"/>
   </link>
-<joint name="lense_box" type="fixed">
+<joint name="lense_box" type="prismatic">
     <parent link="box"/>
     <child link="lense"/>
+    <limit effort="1000.0" lower="0.38" upper="0" velocity="0.5"/>
     <origin xyz="0 0 0" rpy="0 0 0" />
   </joint>
